File: PCBs/input-selector.brd (EAGLE design)
At the start: 84.8 x 48.3 mm, 46 parts, among them IC1 MCP23S17SO, IC2 ULN2803, IC3 ULN2803, K1 AGQ2104H, K2 AGQ2104H, K3 AGQ2104H, K4 AGQ2104H, K5 AGQ2104H, K6 AGQ2104H

Commit message: Initial commit with first changes
Parts:
- removed IN4, IN5: (no value), con-molex:22-23-2031
- removed K4, K5: AGQ2104H, panasonic-agq:PCBBOARD
- removed R10, R11, R12, R7, R8, R9: 47R, rcl:R1206
- added MUTE_IN2: (no value), con-molex:22-23-2031
- moved SEL_OUT 26.1 mm to (37.1, 41.9)
- turned MUTE_OUT2 to 0 degrees
- renumbered IN6 to MUTE_OUT2, K6 to KMUTE2, KMUTE to KMUTE1, MUTE_IN to MUTE_IN1, MUTE_OUT to MUTE_OUT1
Connections:
- removed net N$26: IN5.1, K5.4
- removed net N$27: IN5.3, K5.5
- removed net N$28: KMUTE2.4, MUTE_OUT2.1
- removed net N$29: KMUTE2.5, MUTE_OUT2.3
- removed net N$35: IN4.1, K4.4
- removed net N$36: IN4.3, K4.5
- new net N$20: KMUTE2.6, MUTE_OUT2.3
- new net N$24: KMUTE2.3, MUTE_OUT2.1
- new net OUTL1: KMUTE2.4, MUTE_IN2.1
- new net OUTR1: KMUTE2.5, MUTE_IN2.3
- net +5V: now also KMUTE2.8; no longer R10.1, R11.1, R12.1, R7.1, R8.1, R9.1
- net AGND: now also KMUTE2.2, KMUTE2.7, MUTE_IN2.2; no longer IN4.2, IN5.2
- net INL: no longer K4.3, K5.3, KMUTE2.3
- net INR: no longer K4.6, K5.6, KMUTE2.6
- net N$11: no longer K4.1, R8.2
- net N$13: no longer K3.8, R5.2
- net N$14: now also K3.8, R5.2; no longer K3.1, R6.2
- net N$15: no longer K5.8, R9.2
- net N$16: no longer KMUTE2.8, R11.2
- net N$19: no longer R12.2
- net N$22: now also K3.1, R6.2; no longer K4.8, R7.2
- net N$23: no longer K5.1, R10.2
Routing:
- net INR: track 74.2 -> 34.3 mm
- net INL: track 72.8 -> 35.8 mm
- net +5V: track 173.6 -> 147.4 mm
- net N$23: track 8.57 -> 0.00 mm
- net N$11: track 8.15 -> 0.00 mm
- net N$15: track 7.41 -> 0.00 mm
- net N$36: track 5.00 -> 0.00 mm
- net N$35: track 5.00 -> 0.00 mm
- net N$29: track 5.00 -> 0.00 mm
- net N$28: track 5.00 -> 0.00 mm
- net N$27: track 5.00 -> 0.00 mm
- net N$26: track 5.00 -> 0.00 mm
- net N$13: track 10.5 -> 7.14 mm
- net N$19: track 14.3 -> 11.2 mm
- net N$16: track 10.6 -> 7.55 mm
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
Commit message: Finished up connections
Parts:
- removed EXTRA_IO: 22-23-2031, con-molex:22-23-2031
- added EXT-RELAY, EXT-RELAY1: EXT-RELAY, SparkFun-Connectors:MOLEX-1X4
- turned MUTE_OUT2 to 180 degrees
Connections:
- net +5V: now also KMUTE2.1; no longer KMUTE2.8
- net N$10: now also EXT-RELAY1.3, IC3.17; no longer EXTRA_IO.1, IC3.18
- net N$11: now also EXT-RELAY.1
- net N$12: now also IC3.11; no longer IC3.12
- net N$13: now also EXT-RELAY1.4, IC3.18; no longer IC3.11
- net N$15: now also EXT-RELAY.2
- net N$16: now also EXT-RELAY.4
- net N$19: now also KMUTE2.8; no longer KMUTE2.1
- net N$2: now also EXT-RELAY1.1, IC3.15; no longer EXTRA_IO.2, IC3.17
- net N$23: now also EXT-RELAY.3
- net N$4: now also EXT-RELAY1.2; no longer EXTRA_IO.3
- net N$5: now also IC3.14; no longer IC3.15
- net N$8: now also IC3.13; no longer IC3.14
- net N$9: now also IC3.12; no longer IC3.13
Routing:
- net N$11: track 0.00 -> 38.6 mm
- net N$15: track 0.00 -> 36.1 mm
- net N$23: track 0.00 -> 34.1 mm
- net N$16: track 7.55 -> 33.8 mm
- net +5V: track 147.4 -> 167.9 mm
- net OUTL1: track 0.00 -> 16.7 mm
- net OUTR1: track 0.00 -> 13.3 mm
- net N$24: track 0.00 -> 8.37 mm
- net N$20: track 0.00 -> 8.19 mm
- net N$14: track 11.9 -> 17.6 mm
- net N$19: track 11.2 -> 6.80 mm
- net N$22: track 10.3 -> 14.4 mm
- net N$2: track 12.5 -> 16.1 mm
- net N$9: track 7.41 -> 4.83 mm
- net N$10: track 10.0 -> 11.7 mm
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Other:
- board text added: "EXTRA_IO"
- board text added: "EXT_RELAYS"
- board text removed: "Designed by Max Williams"
