File: PCBs/input-selector.sch (EAGLE design)
At the start: 39 parts, among them IC1 MCP23S17SO, IC2 ULN2803, IC3 ULN2803, K1 AGQ2104H, K2 AGQ2104H, K3 AGQ2104H, K4 AGQ2104H, K5 AGQ2104H, K6 AGQ2104H

Commit message: Initial commit with first changes
Parts:
- removed IN4, IN5, IN6, MUTE_IN: 22-23-2031, con-molex:22-23-2031
- removed K4, K5, K6, KMUTE: AGQ2104H, panasonic-agq:AGQ2104H
- removed R10, R11, R12, R7, R8, R9: 47R, rcl:R-EU_R1206
- added KMUTE1, KMUTE2: AGQ2104H, panasonic-agq:AGQ2104H
- added MUTE_IN1, MUTE_IN2, MUTE_OUT2: 22-23-2031, con-molex:22-23-2031
- renumbered MUTE_OUT to MUTE_OUT1
Connections:
- removed net N$26: IN5-1.S, K5G$3.S
- removed net N$27: IN5-3.S, K5G$2.S
- removed net N$28: IN6-1.S, K6G$3.S
- removed net N$29: IN6-3.S, K6G$2.S
- removed net N$35: IN4-1.S, K4G$3.S
- removed net N$36: IN4-3.S, K4G$2.S
- new net N$20: KMUTE2G$2.P, MUTE_OUT2-3.S
- new net N$24: KMUTE2G$3.P, MUTE_OUT2-1.S
- new net OUTL1: KMUTE2G$3.S, MUTE_IN2-1.S
- new net OUTR1: KMUTE2G$2.S, MUTE_IN2-3.S
- net +5V: now also KMUTE1G$1.+, KMUTE2G$1.-; no longer KMUTEG$1.+, R10.1, R11.1, R12.1, R7.1, R8.1, R9.1
- net AGND: now also KMUTE1G$2.O, KMUTE1G$3.O, KMUTE2G$2.O, KMUTE2G$3.O, MUTE_IN1-2.S, MUTE_IN2-2.S, MUTE_OUT2-2.S; no longer IN4-2.S, IN5-2.S, IN6-2.S, KMUTEG$2.O, KMUTEG$3.O, MUTE_IN-2.S
- net INL: no longer K4G$3.P, K5G$3.P, K6G$3.P
- net INR: no longer K4G$2.P, K5G$2.P, K6G$2.P
- net N$11: no longer K4G$1.+, R8.2
- net N$13: no longer K3G$1.-, R5.2
- net N$14: now also K3G$1.-, R5.2; no longer K3G$1.+, R6.2
- net N$15: no longer K5G$1.-, R9.2
- net N$16: no longer K6G$1.-, R11.2
- net N$17: now also KMUTE1G$2.P; no longer KMUTEG$2.P
- net N$18: now also KMUTE1G$3.P; no longer KMUTEG$3.P
- net N$19: now also KMUTE2G$1.+; no longer K6G$1.+, R12.2
- net N$22: now also K3G$1.+, R6.2; no longer K4G$1.-, R7.2
- net N$23: no longer K5G$1.+, R10.2
- net N$6: now also KMUTE1G$1.-; no longer KMUTEG$1.-
- net OUTL: now also KMUTE1G$3.S, MUTE_IN1-1.S; no longer KMUTEG$3.S, MUTE_IN-1.S
- net OUTR: now also KMUTE1G$2.S, MUTE_IN1-3.S; no longer KMUTEG$2.S, MUTE_IN-3.S
Other:
- moved on the sheet: IN2-1, IN2-2, IN2-3, IN3-1, IN3-2, IN3-3, K2, K3

Commit message: Finished up connections
Parts:
- removed EXTRA_IO: 22-23-2031, con-molex:22-23-2031
- added EXT-RELAY, EXT-RELAY1: EXT-RELAY, SparkFun-Connectors:M04POLAR
Connections:
- net +5V: now also KMUTE2G$1.+; no longer KMUTE2G$1.-
- net N$10: now also EXT-RELAY1.3, IC3.O2; no longer EXTRA_IO-1.S, IC3.O1
- net N$11: now also EXT-RELAY.1
- net N$12: now also IC3.O8; no longer IC3.O7
- net N$13: now also EXT-RELAY1.4, IC3.O1; no longer IC3.O8
- net N$15: now also EXT-RELAY.2
- net N$16: now also EXT-RELAY.4
- net N$19: now also KMUTE2G$1.-; no longer KMUTE2G$1.+
- net N$2: now also EXT-RELAY1.1, IC3.O4; no longer EXTRA_IO-2.S, IC3.O2
- net N$23: now also EXT-RELAY.3
- net N$4: now also EXT-RELAY1.2; no longer EXTRA_IO-3.S
- net N$5: now also IC3.O5; no longer IC3.O4
- net N$8: now also IC3.O6; no longer IC3.O5
- net N$9: now also IC3.O7; no longer IC3.O6
Other:
- moved on the sheet: K1, K2, KMUTE2, R1, R2, R3, R4
